File: hardware/atmega32u4-dev.kicad_pcb (KiCad board)
At the start: 2 copper layers, 45.7 x 20.3 mm, 70 parts, among them J1 Conn_01x02_Male, J2 USB_C_Receptacle_USB2.0, J3 Conn_01x14, J4 Conn_01x14, Q1 AO3401A, U1 LTC4054ES5-4.2, U2 AP2112K-3.3, U3 ATmega32U4-M, Y1 Resonator

Commit message: Generated BOM and fabrication files for v1.0.0 boards.
Changed lines of the file:
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@@
       (layerselection 0x00010fc_ffffffff)
       (disableapertmacros false)
-      (usegerberextensions false)
+      (usegerberextensions true)
       (usegerberattributes true)
       (usegerberadvancedattributes true)
-      (creategerberjobfile true)
+      (creategerberjobfile false)
       (svguseinch false)
       (svgprecision 6)
@@
       (psa4output false)
       (plotreference true)
-      (plotvalue true)
+      (plotvalue false)
       (plotinvisibletext false)
       (sketchpadsonfab false)
-      (subtractmaskfromsilk false)
+      (subtractmaskfromsilk true)
       (outputformat 1)
       (mirror false)
-      (drillshape 1)
+      (drillshape 0)
       (scaleselection 1)
-      (outputdirectory "")
+      (outputdirectory "fabrication/")
     )
   )
@@
     (fp_line (start -2.5 -3.5) (end 3.5 -3.5) (layer "F.Fab") (width 0.1))
     (fp_line (start -3.5 3.5) (end -3.5 -2.5) (layer "F.Fab") (width 0.1))
-    (pad "" smd roundrect locked (at -0.65 -0.65 225) (size 1.05 1.05) (layers "F.Paste") (roundrect_rratio 0.238095))
-    (pad "" smd roundrect locked (at 0.65 -1.95 225) (size 1.05 1.05) (layers "F.Paste") (roundrect_rratio 0.238095))
-    (pad "" smd roundrect locked (at -1.95 -1.95 225) (size 1.05 1.05) (layers "F.Paste") (roundrect_rratio 0.238095))
-    (pad "" smd roundrect locked (at -1.95 1.95 225) (size 1.05 1.05) (layers "F.Paste") (roundrect_rratio 0.238095))
-    (pad "" smd roundrect locked (at 0.65 1.95 225) (size 1.05 1.05) (layers "F.Paste") (roundrect_rratio 0.238095))
-    (pad "" smd roundrect locked (at 1.95 1.95 225) (size 1.05 1.05) (layers "F.Paste") (roundrect_rratio 0.238095))
-    (pad "" smd roundrect locked (at 0.65 -0.65 225) (size 1.05 1.05) (layers "F.Paste") (roundrect_rratio 0.238095))
-    (pad "" smd roundrect locked (at 1.95 -0.65 225) (size 1.05 1.05) (layers "F.Paste") (roundrect_rratio 0.238095))
-    (pad "" smd roundrect locked (at 1.95 0.65 225) (size 1.05 1.05) (layers "F.Paste") (roundrect_rratio 0.238095))
-    (pad "" smd roundrect locked (at -1.95 -0.65 225) (size 1.05 1.05) (layers "F.Paste") (roundrect_rratio 0.238095))
-    (pad "" smd roundrect locked (at -0.65 0.65 225) (size 1.05 1.05) (layers "F.Paste") (roundrect_rratio 0.238095))
-    (pad "" smd roundrect locked (at 0.65 0.65 225) (size 1.05 1.05) (layers "F.Paste") (roundrect_rratio 0.238095))
-    (pad "" smd roundrect locked (at -0.65 1.95 225) (size 1.05 1.05) (layers "F.Paste") (roundrect_rratio 0.238095))
-    (pad "" smd roundrect locked (at -1.95 0.65 225) (size 1.05 1.05) (layers "F.Paste") (roundrect_rratio 0.238095))
-    (pad "" smd roundrect locked (at -0.65 -1.95 225) (size 1.05 1.05) (layers "F.Paste") (roundrect_rratio 0.238095))
-    (pad "" smd roundrect locked (at 1.95 -1.95 225) (size 1.05 1.05) (layers "F.Paste") (roundrect_rratio 0.238095))
+    (pad "" smd roundrect locked (at -0.65 -0.65 225) (size 1.05 1.05) (layers "F.Paste") (roundrect_rratio 0.2380952381))
+    (pad "" smd roundrect locked (at 0.65 -1.95 225) (size 1.05 1.05) (layers "F.Paste") (roundrect_rratio 0.2380952381))
+    (pad "" smd roundrect locked (at -1.95 -1.95 225) (size 1.05 1.05) (layers "F.Paste") (roundrect_rratio 0.2380952381))
+    (pad "" smd roundrect locked (at -1.95 1.95 225) (size 1.05 1.05) (layers "F.Paste") (roundrect_rratio 0.2380952381))
+    (pad "" smd roundrect locked (at 0.65 1.95 225) (size 1.05 1.05) (layers "F.Paste") (roundrect_rratio 0.2380952381))
+    (pad "" smd roundrect locked (at 1.95 1.95 225) (size 1.05 1.05) (layers "F.Paste") (roundrect_rratio 0.2380952381))
+    (pad "" smd roundrect locked (at 0.65 -0.65 225) (size 1.05 1.05) (layers "F.Paste") (roundrect_rratio 0.2380952381))
+    (pad "" smd roundrect locked (at 1.95 -0.65 225) (size 1.05 1.05) (layers "F.Paste") (roundrect_rratio 0.2380952381))
+    (pad "" smd roundrect locked (at 1.95 0.65 225) (size 1.05 1.05) (layers "F.Paste") (roundrect_rratio 0.2380952381))
+    (pad "" smd roundrect locked (at -1.95 -0.65 225) (size 1.05 1.05) (layers "F.Paste") (roundrect_rratio 0.2380952381))
+    (pad "" smd roundrect locked (at -0.65 0.65 225) (size 1.05 1.05) (layers "F.Paste") (roundrect_rratio 0.2380952381))
+    (pad "" smd roundrect locked (at 0.65 0.65 225) (size 1.05 1.05) (layers "F.Paste") (roundrect_rratio 0.2380952381))
+    (pad "" smd roundrect locked (at -0.65 1.95 225) (size 1.05 1.05) (layers "F.Paste") (roundrect_rratio 0.2380952381))
+    (pad "" smd roundrect locked (at -1.95 0.65 225) (size 1.05 1.05) (layers "F.Paste") (roundrect_rratio 0.2380952381))
+    (pad "" smd roundrect locked (at -0.65 -1.95 225) (size 1.05 1.05) (layers "F.Paste") (roundrect_rratio 0.2380952381))
+    (pad "" smd roundrect locked (at 1.95 -1.95 225) (size 1.05 1.05) (layers "F.Paste") (roundrect_rratio 0.2380952381))
     (pad "1" smd roundrect locked (at -3.3375 -2.5 225) (size 1.075 0.25) (layers "F.Cu" "F.Paste" "F.Mask") (roundrect_rratio 0.25)
       (net 25 "/D7") (pinfunction "PE6") (pintype "bidirectional"))
@@
     (fp_line (start 0 0.875) (end -0.5 1.375) (layer "F.Fab") (width 0.1))
     (fp_line (start 3.25 0.25) (end -1.25 0.25) (layer "F.Fab") (width 0.1))
-    (pad "1" thru_hole roundrect locked (at 0 0 90) (size 1.2 1.75) (drill 0.75) (layers *.Cu *.Mask) (roundrect_rratio 0.208333)
+    (pad "1" thru_hole roundrect locked (at 0 0 90) (size 1.2 1.75) (drill 0.75) (layers *.Cu *.Mask) (roundrect_rratio 0.2083333333)
       (net 5 "+BATT") (pinfunction "Pin_1") (pintype "passive"))
     (pad "2" thru_hole oval locked (at 2 0 90) (size 1.2 1.75) (drill 0.75) (layers *.Cu *.Mask)
