File: hardware/atmega32u4-dev.kicad_sch (KiCad schematic)
At the start: 43 parts, among them J1 Conn_01x02_Male, J2 USB_C_Receptacle_USB2.0, J3 Conn_01x14, J4 Conn_01x14, Q1 AO3400A, Q2 AO3401A, SW1 SW_SPST, SW2 SW_SPST, U1 LTC4054ES5-4.2, U2 AP2112K-3.3, U3 ATmega32U4-M, Y1 Resonator

Commit message: Completed PCB layout
Completed PCB layout for manufacture.
Parts:
- removed L1: 10uH, Inductor_SMD:L_0603_1608Metric, symbol Device:L
- removed Q1: AO3400A, Package_TO_SOT_SMD:SOT-23, symbol Transistor_FET:AO3400A
- removed R1: 100k, Resistor_SMD:R_0603_1608Metric, symbol Device:R
- removed R12, R13, R14, R15: 100, Resistor_SMD:R_0603_1608Metric, symbol Device:R
- removed R7: 1, Resistor_SMD:R_0603_1608Metric, symbol Device:R
- removed SW1, SW2: SW_SPST, Button_Switch_SMD:SW_SPST_TL3342, symbol Switch:SW_SPST
- added C2: 10uF, Capacitor_SMD:C_0603_1608Metric, symbol Device:C
- renumbered C9 to C10, C2 to C3, C3 to C4, C4 to C5, C5 to C6, C6 to C7, C7 to C8, C8 to C9, Q2 to Q1, R2 to R1, R3 to R2, R4 to R3, R5 to R4, R6 to R5, R8 to R6, R9 to R7, R10 to R8, R11 to R9
Connections:
- net +3V3: now also C10.1, D6.2 (A), J4.6 (Pin_6), U3.24 (AVCC), U3.44 (AVCC)
- net A0: now also J3.9 (Pin_9)
- net A1: now also J3.10 (Pin_10)
- net A2: now also J3.11 (Pin_11)
- net A3: now also J3.12 (Pin_12)
- net A4: now also J3.13 (Pin_13)
- net A5: now also J3.14 (Pin_14)
- net D10: now also J3.7 (Pin_7)
- net D11: now also J4.8 (Pin_8)
- net D12: now also J4.9 (Pin_9)
- net D13: now also D3.2 (A), J4.10 (Pin_10)
- net D4: now also J3.1 (Pin_1)
- net D5: now also J3.2 (Pin_2)
- net D6: now also J3.3 (Pin_3)
- net D7: now also J3.4 (Pin_4)
- net D8: now also J3.5 (Pin_5)
- net D9: now also J3.6 (Pin_6)
- net GND: now also C5.1, J3.8 (Pin_8), R2.2, C2.2
- net HWB: now also J4.5 (Pin_5)
- net MISO: now also J4.11 (Pin_11)
- net MOSI: now also J4.12 (Pin_12)
- net RST: now also J4.7 (Pin_7)
- net RX: now also J4.2 (Pin_2)
- net RXLED: now also D4.2 (A)
- net SCK: now also J4.13 (Pin_13)
- net SCL: now also J4.4 (Pin_4)
- net SDA: now also J4.3 (Pin_3)
- net TX: now also J4.1 (Pin_1)
- net TXLED: now also D5.2 (A)
- net VBUS: now also C2.1
- net Vin: now also J4.14 (Pin_14)
- net U_P: now reaches R6.2, U3.4 (D+)
- net U_N: now reaches R7.2, U3.3 (D-)
- no-connect marks 32 -> 4
Other:
- moved on the sheet: C1, C9, R2

Commit message: Completed v1.0.0
Added files for LiPo boost and motor driver board. Completed schematic and layout.
Other:
- title: ATmega32u4 Development Board -> ATmega32u4 Development Micro Board
Changed lines of the file:
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@@
   (paper "A4")
   (title_block
-    (title "ATmega32u4 Development Board")
-    (date "2023-02-23")
+    (title "ATmega32u4 Development Micro Board")
+    (date "2023-05-28")
     (rev "v1.0.0")
     (company "Shadman Habib")

Commit message: Generated BOM and fabrication files for v1.0.0 boards.
Parts:
- J1, J3, J4: now left out of the parts list
Changed lines of the file:
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@@
   )
   (symbol (lib_id "Connector_Generic:Conn_01x14") (at 231.14 127 0) (unit 1)
-    (in_bom yes) (on_board yes) (fields_autoplaced)
+    (in_bom no) (on_board yes) (fields_autoplaced)
     (property "Reference" "J3" (id 0) (at 231.14 148.59 0))
     (property "Value" "Conn_01x14" (id 1) (at 231.14 151.13 0))
@@
   )
   (symbol (lib_id "Connector:Conn_01x02_Male") (at 25.4 158.75 0) (unit 1)
-    (in_bom yes) (on_board yes) (fields_autoplaced)
+    (in_bom no) (on_board yes) (fields_autoplaced)
     (property "Reference" "J1" (id 0) (at 26.035 156.21 0))
     (property "Value" "Conn_01x02_Male" (id 1) (at 26.035 156.21 0)
@@
   (symbol (lib_id "power:+3.3V") (at 204.47 46.99 0) (unit 1)
     (in_bom yes) (on_board yes) (fields_autoplaced)
-    (property "Reference" "#PWR029" (id 0) (at 204.47 50.8 0)
+    (property "Reference" "#PWR028" (id 0) (at 204.47 50.8 0)
       (effects (font (size 1.27 1.27)) hide)
     )
@@
   (symbol (lib_id "power:GND") (at 213.36 129.54 270) (unit 1)
     (in_bom yes) (on_board yes) (fields_autoplaced)
-    (property "Reference" "#PWR0101" (id 0) (at 207.01 129.54 0)
+    (property "Reference" "#PWR029" (id 0) (at 207.01 129.54 0)
       (effects (font (size 1.27 1.27)) hide)
     )
@@
   (symbol (lib_id "power:+3.3V") (at 245.11 76.2 0) (unit 1)
     (in_bom yes) (on_board yes) (fields_autoplaced)
-    (property "Reference" "#PWR031" (id 0) (at 245.11 80.01 0)
+    (property "Reference" "#PWR030" (id 0) (at 245.11 80.01 0)
       (effects (font (size 1.27 1.27)) hide)
     )
@@
   )
   (symbol (lib_id "Connector_Generic:Conn_01x14") (at 241.3 127 0) (mirror y) (unit 1)
-    (in_bom yes) (on_board yes) (fields_autoplaced)
+    (in_bom no) (on_board yes) (fields_autoplaced)
     (property "Reference" "J4" (id 0) (at 241.3 105.41 0))
     (property "Value" "Conn_01x14" (id 1) (at 241.3 107.95 0))
@@
   (symbol (lib_id "power:+3.3V") (at 259.08 124.46 270) (unit 1)
     (in_bom yes) (on_board yes) (fields_autoplaced)
-    (property "Reference" "#PWR?" (id 0) (at 255.27 124.46 0)
+    (property "Reference" "#PWR031" (id 0) (at 255.27 124.46 0)
       (effects (font (size 1.27 1.27)) hide)
     )
@@
     )
     (path "/641c6658-c79b-48e6-988c-a2dfa5ba8ca3"
-      (reference "#PWR029") (unit 1) (value "+3.3V") (footprint "")
+      (reference "#PWR028") (unit 1) (value "+3.3V") (footprint "")
+    )
+    (path "/731ff3e5-4523-4edc-beb4-548e26fedcf4"
+      (reference "#PWR029") (unit 1) (value "GND") (footprint "")
     )
     (path "/c666ad59-31f7-4347-96ad-fb15f56ed6a1"
+      (reference "#PWR030") (unit 1) (value "+3.3V") (footprint "")
+    )
+    (path "/e68543c7-4374-4560-bf9e-80062f46e69a"
       (reference "#PWR031") (unit 1) (value "+3.3V") (footprint "")
     )
@@
       (reference "#PWR032") (unit 1) (value "GND") (footprint "")
     )
-    (path "/731ff3e5-4523-4edc-beb4-548e26fedcf4"
-      (reference "#PWR0101") (unit 1) (value "GND") (footprint "")
-    )
-    (path "/e68543c7-4374-4560-bf9e-80062f46e69a"
-      (reference "#PWR?") (unit 1) (value "+3.3V") (footprint "")
-    )
     (path "/845cb57f-abd1-4d78-9b0b-4e675805ee06"
